Commit message: fix

File: source/tactile_tasks/assets/urdf/allegro_hand_right.urdf (robot description, URDF)
Before this commit: robot hand_object, 25 links, 24 joints
Links:
- link hitosashi_ee: geometry collision sphere radius=0.005; visual sphere radius=0.005
- link kusuri_ee: geometry collision sphere radius=0.005; visual sphere radius=0.005
- link naka_ee: geometry collision sphere radius=0.005; visual sphere radius=0.005
- link oya_ee: geometry collision sphere radius=0.005; visual sphere radius=0.005
