Commit message: changed sd geometry, added internal env noise

File: source/tactile_tasks/assets/urdf/screwdriver/screwdriver_free.urdf (robot description, URDF)
Before this commit: robot screwdriver_on_the_table, 2 links, 1 joints
Links:
- link screwdriver_body: geometry collision cylinder length=0.1 radius=0.0175; visual cylinder length=0.1 radius=0.0175
